File: schematic/race_4_players/race_4_players.kicad_sch (KiCad schematic)
At the start: 8 parts, among them SW1 Red_Push, SW2 Blue_Push, SW3 Green_Push, SW4 Yellow_Push

Commit message: update schematic (include de0 nano mini header)
Connections:
- net blue_input: no longer SW2.2
- net green_input: no longer SW3.2
- net red_input: no longer SW1.2
- net yellow_input: no longer SW4.2
Other:
- added sheet de0_nano_mini (de0_nano_mini.kicad_sch)
Changed lines of the file:
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@@
 	(generator_version "8.0")
 	(paper "A4")
-	(junction
-		(at 219.71 57.15)
-		(diameter 0)
-		(color 0 0 0 0)
-	)
-	(junction
-		(at 114.3 99.06)
-		(diameter 0)
-		(color 0 0 0 0)
-	)
-	(junction
-		(at 218.44 99.06)
-		(diameter 0)
-		(color 0 0 0 0)
-	)
-	(junction
-		(at 114.3 54.61)
-		(diameter 0)
-		(color 0 0 0 0)
-	)
 	(wire
 		(pts
@@
 	(wire
 		(pts
-			(xy 219.71 57.15) (xy 227.33 57.15)
-		)
-		(stroke
-			(width 0)
-			(type default)
-		)
-	)
-	(wire
-		(pts
-			(xy 87.63 54.61) (xy 114.3 54.61)
+			(xy 87.63 54.61) (xy 123.19 54.61)
 		)
 		(stroke
@@
 	(wire
 		(pts
-			(xy 191.77 99.06) (xy 218.44 99.06)
+			(xy 191.77 99.06) (xy 226.06 99.06)
 		)
 		(stroke
@@
 	(wire
 		(pts
-			(xy 218.44 99.06) (xy 226.06 99.06)
-		)
-		(stroke
-			(width 0)
-			(type default)
-		)
-	)
-	(wire
-		(pts
 			(xy 196.85 80.01) (xy 196.85 91.44)
 		)
@@
 	(wire
 		(pts
-			(xy 193.04 57.15) (xy 219.71 57.15)
+			(xy 193.04 57.15) (xy 227.33 57.15)
 		)
 		(stroke
@@
 	(wire
 		(pts
-			(xy 114.3 54.61) (xy 123.19 54.61)
-		)
-		(stroke
-			(width 0)
-			(type default)
-		)
-	)
-	(wire
-		(pts
 			(xy 173.99 99.06) (xy 173.99 109.22)
 		)
@@
 	(wire
 		(pts
-			(xy 90.17 99.06) (xy 114.3 99.06)
+			(xy 90.17 99.06) (xy 123.19 99.06)
 		)
 		(stroke
@@
 		(pts
 			(xy 173.99 99.06) (xy 184.15 99.06)
-		)
-		(stroke
-			(width 0)
-			(type default)
-		)
-	)
-	(wire
-		(pts
-			(xy 114.3 99.06) (xy 123.19 99.06)
 		)
 		(stroke
@@
 				)
 			)
+		)
+	)
+	(sheet
+		(at 1.27 237.49)
+		(size 297.18 238.76)
+		(fields_autoplaced yes)
+		(stroke
+			(width 0.1524)
+			(type solid)
+		)
+		(fill
+			(color 0 0 0 0.0000)
+		)
+		(property "Sheetname" "de0_nano_mini"
+			(at 1.27 236.7784 0)
+			(effects
+				(font
+					(size 1.27 1.27)
+				)
+				(justify left bottom)
+			)
+		)
+		(property "Sheetfile" "de0_nano_mini.kicad_sch"
+			(at 1.27 476.8346 0)
+			(effects
+				(font
+					(size 1.27 1.27)
+				)
+				(justify left top)
+			)
+		)
+		(instances
+			(project "race_4_players"
+				(path "/40e8b58e-fede-4956-ac8c-a3df9c5062b3"
+					(page "2")
+				)
+			)
